File: Arduino Clone - BACEE.sch (KiCad schematic (older format))
At the start: 13 parts, among them U1 24LC1025, U2 24LC1025, U3 DS13375+, U4 ATMEGA328P-AU, Y1 Crystal 32Mhz, Y2 Crystal 16Mhz

Commit message: wiring
Parts:
- removed BT1: Battery 3V, Connector_PinHeader_2.54mm:PinHeader_1x02_P2.54mm_Vertical, symbol Device:Battery
- removed C3: 10uF, Capacitor_SMD:C_0805_2012Metric_Pad1.15x1.40mm_HandSolder, symbol Device:CP
- added BT?: Battery 3V, Connector_PinHeader_2.54mm:PinHeader_1x02_P2.54mm_Vertical, symbol Device:Battery
- added C?: 10uF, Capacitor_SMD:C_0805_2012Metric_Pad1.15x1.40mm_HandSolder, symbol Device:CP
Connections:
- net GND is gone; now on net GNDPWR: U4.21 (GND), U4.3 (GND), U4.5 (GND)
- net RESET: now also R2.1
- net SCK: now also D1.2 (A), U1.6 (SCL), U2.6 (SCL), U3.6 (SCL)
- net SDA: now also U1.5 (SDA), U2.5 (SDA), U3.5 (SDA)
- net Vcc: now also R2.2, U1.3 (A2), U1.8 (VCC), U2.3 (A2), U2.8 (VCC), U3.3 (INTA), U3.8 (Vcc), U4.20 (AREF), BT?.1 (+), C?.1
- net GNDPWR: now reaches C1.1
- net GNDPWR: now also C2.1, R1.2, U1.4 (GND), U1.7 (WP), U2.4 (GND), U2.7 (WP), U3.4 (GND), BT?.2 (-), C?.2
- net at C1.2: now also U4.7 (PB6), Y2.1
- net at C2.2: now also U4.8 (PB7), Y2.2
- net at D1.1 (K): now also R1.1
- net ADDS1: now reaches U1.1 (A0)
- net ADDS1: now also U2.1 (A0), U4.23 (PC0)
- net ADDS2: now reaches U1.2 (A1)
- net ADDS2: now also U2.2 (A1), U4.24 (PC1)
- net at U3.1 (X1): now also Y1.1, Y1.2
- no-connect marks 0 -> 7
Other:
- moved on the sheet: C2, D1, R1, R2, U2, U3, Y1

Commit message: ERC
Parts:
- gave numbers to parts that had none: 2
Connections:
- net at U3.1 (X1), Y1.2: no longer Y1.1
- net at U3.2 (X2): now also Y1.1
- no-connect marks 7 -> 8
Changed lines of the file:
@@
 	6000 5650 6000 5750
 $Comp
-L power:GNDPWR #PWR?
+L power:GNDPWR #PWR0101
 U 1 1 5E90B31A
 P 5000 7400
-F 0 "#PWR?" H 5000 7200 50  0001 C CNN
+F 0 "#PWR0101" H 5000 7200 50  0001 C CNN
 F 1 "GNDPWR" H 5004 7246 50  0000 C CNN
 F 2 "" H 5000 7350 50  0001 C CNN
@@
 Wire Wire Line
 	2600 2100 2700 2100
-Wire Wire Line
-	2600 2100 2600 2150
-Wire Wire Line
-	2600 2150 2400 2150
-Wire Wire Line
-	2400 2150 2400 2250
-Wire Wire Line
-	2400 2250 2250 2250
-Connection ~ 2600 2100
-$Comp
-L power:GNDPWR #PWR?
+$Comp
+L power:GNDPWR #PWR0102
 U 1 1 5E91C1AD
 P 3200 2800
-F 0 "#PWR?" H 3200 2600 50  0001 C CNN
+F 0 "#PWR0102" H 3200 2600 50  0001 C CNN
 F 1 "GNDPWR" H 3204 2646 50  0000 C CNN
 F 2 "" H 3200 2750 50  0001 C CNN
@@
 	2600 5650 3150 5650
 $Comp
-L power:GNDPWR #PWR?
+L power:GNDPWR #PWR0103
 U 1 1 5E9230AE
 P 2600 5700
-F 0 "#PWR?" H 2600 5500 50  0001 C CNN
+F 0 "#PWR0103" H 2600 5500 50  0001 C CNN
 F 1 "GNDPWR" H 2604 5546 50  0000 C CNN
 F 2 "" H 2600 5650 50  0001 C CNN
@@
 ADDS2
 $Comp
-L power:GNDPWR #PWR?
+L power:GNDPWR #PWR0104
 U 1 1 5E927E27
 P 6750 3600
-F 0 "#PWR?" H 6750 3400 50  0001 C CNN
+F 0 "#PWR0104" H 6750 3400 50  0001 C CNN
 F 1 "GNDPWR" H 6754 3446 50  0000 C CNN
 F 2 "" H 6750 3550 50  0001 C CNN
@@
 $EndComp
 $Comp
-L Device:CP C?
+L Device:CP C3
 U 1 1 5E928BB4
 P 6500 3050
-F 0 "C?" H 6618 3096 50  0000 L CNN
+F 0 "C3" H 6618 3096 50  0000 L CNN
 F 1 "10uF" H 6618 3005 50  0000 L CNN
 F 2 "Capacitor_SMD:C_0805_2012Metric_Pad1.15x1.40mm_HandSolder" H 6538 2900 50  0001 C CNN
@@
 $EndComp
 $Comp
-L Device:Battery BT?
+L Device:Battery BT1
 U 1 1 5E929089
 P 7050 3100
-F 0 "BT?" H 7158 3146 50  0000 L CNN
+F 0 "BT1" H 7158 3146 50  0000 L CNN
 F 1 "Battery 3V" H 7158 3055 50  0000 L CNN
 F 2 "Connector_PinHeader_2.54mm:PinHeader_1x02_P2.54mm_Vertical" V 7050 3160 50  0001 C CNN
@@
 	6800 2900 7050 2900
 Wire Wire Line
-	6000 2300 6800 2300
+	6000 2300 6350 2300
 Wire Wire Line
 	6800 2300 6800 2900
@@
 Connection ~ 4000 3400
 $Comp
-L power:GNDPWR #PWR?
+L power:GNDPWR #PWR0105
 U 1 1 5E9538E8
 P 4000 3500
-F 0 "#PWR?" H 4000 3300 50  0001 C CNN
+F 0 "#PWR0105" H 4000 3300 50  0001 C CNN
 F 1 "GNDPWR" H 4004 3346 50  0000 C CNN
 F 2 "" H 4000 3450 50  0001 C CNN
@@
 	4700 4050 4700 4150
 $Comp
-L power:GNDPWR #PWR?
+L power:GNDPWR #PWR0106
 U 1 1 5E959FAA
 P 4700 4450
-F 0 "#PWR?" H 4700 4250 50  0001 C CNN
+F 0 "#PWR0106" H 4700 4250 50  0001 C CNN
 F 1 "GNDPWR" H 4704 4296 50  0000 C CNN
 F 2 "" H 4700 4400 50  0001 C CNN
@@
 GND
 $Comp
-L power:GNDPWR #PWR?
+L power:GNDPWR #PWR0107
 U 1 1 5E95F7E3
 P 6000 5750
-F 0 "#PWR?" H 6000 5550 50  0001 C CNN
+F 0 "#PWR0107" H 6000 5550 50  0001 C CNN
 F 1 "GNDPWR" H 6004 5596 50  0000 C CNN
 F 2 "" H 6000 5700 50  0001 C CNN
@@
 NoConn ~ 5400 5150
 NoConn ~ 5400 5350
+NoConn ~ 5400 4650
+Wire Wire Line
+	2250 2250 2700 2250
+$Comp
+L power:PWR_FLAG #FLG0101
+U 1 1 5E96FCF1
+P 6350 2300
+F 0 "#FLG0101" H 6350 2375 50  0001 C CNN
+F 1 "PWR_FLAG" H 6350 2473 50  0000 C CNN
+F 2 "" H 6350 2300 50  0001 C CNN
+F 3 "~" H 6350 2300 50  0001 C CNN
+	1    6350 2300
+	1    0    0    -1
+$EndComp
+Connection ~ 6350 2300
+Wire Wire Line
+	6350 2300 6800 2300
 $EndSCHEMATC

Commit message: Comments
Other:
- note added: "N1 - Clock/Calendar\n"
- note added: "N2 - Atmega 328p- au with Oscillator and battery"
- note added: "N3 - EEPROM\n"
- note added: "N4 - Connectors"
- moved on the sheet: BT1, C1, C2, C3, D1, R1, R2, U1, U2, U3, U4, Y1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
