File: Arduino Clone - BACEE.kicad_pcb (KiCad board)
At the start: 2 copper layers, 0 parts

Commit message: Set Design Rules
Parts:
- added BT1: Battery 3V, Connector_PinHeader_2.54mm:PinHeader_1x02_P2.54mm_Vertical, F.Cu at (113.0, 65.4)
- added C1: 22pF, Capacitor_SMD:C_0805_2012Metric_Pad1.15x1.40mm_HandSolder, F.Cu at (160.6, 89.3)
- added C2: 22pF, Capacitor_SMD:C_0805_2012Metric_Pad1.15x1.40mm_HandSolder, F.Cu at (160.7, 95.2)
- added C3: 10uF, Capacitor_SMD:C_0805_2012Metric_Pad1.15x1.40mm_HandSolder, F.Cu at (154.5, 99.5)
- added D1: LED, LED_SMD:LED_0805_2012Metric_Pad1.15x1.40mm_HandSolder, F.Cu at (149.8, 98.4)
- added J1: Digital Pins, Connector_PinSocket_2.54mm:PinSocket_1x09_P2.54mm_Vertical, F.Cu at (90.7, 63.4)
- added J2: Serial, Connector_PinSocket_2.54mm:PinSocket_1x04_P2.54mm_Vertical, F.Cu at (99.9, 62.8)
- added J3: ICSP, Connector_PinSocket_2.54mm:PinSocket_2x03_P2.54mm_Vertical, F.Cu at (107.1, 62.8)
- added J4: I2C, Connector_PinSocket_2.54mm:PinSocket_1x04_P2.54mm_Vertical, F.Cu at (95.3, 62.8)
- added R1: 330Ohms, Resistor_SMD:R_0805_2012Metric_Pad1.15x1.40mm_HandSolder, F.Cu at (160.6, 92.3)
- added R2: 10kOhms, Resistor_SMD:R_0805_2012Metric_Pad1.15x1.40mm_HandSolder, F.Cu at (156.0, 96.5)
- added U1: 24LC1025, Package_SO:SOIJ-8_5.3x5.3mm_P1.27mm, F.Cu at (148.3, 93.4)
- added U2: 24LC1025, Package_SO:SOIJ-8_5.3x5.3mm_P1.27mm, F.Cu at (148.3, 86.5)
- added U3: DS13375+, Package_SO:SO-8_5.3x6.2mm_P1.27mm, F.Cu at (136.9, 98.3)
- added U4: ATMEGA328P-AU, digikey-footprints:TQFP-32_7x7mm, F.Cu at (137.3, 88.7)
- added Y1: Crystal 32Mhz, Crystal:Crystal_SMD_MicroCrystal_CC7V-T1A-2Pin_3.2x1.5mm, F.Cu at (144.8, 98.6)
- added Y2: Crystal 16Mhz, Crystal:Crystal_SMD_5032-2Pin_5.0x3.2mm_HandSoldering, F.Cu at (158.7, 85.4)
Other:
- net class Power added: clearance 0.2, trace_width 0.3, via_dia 1, via_drill 0.6

Commit message: Placement
Parts:
- moved R2 69.0 mm to (87.6, 87.2), turned to 90 degrees
- moved Y2 64.2 mm to (94.6, 87.0)
- moved C2 59.3 mm to (101.8, 88.3)
- moved C1 58.9 mm to (101.8, 85.7)
- moved R1 43.4 mm to (117.7, 99.1)
- moved J1 42.6 mm to (91.4, 106.0), turned to 90 degrees
- moved U4 42.1 mm to (95.9, 96.5)
- moved U1 39.2 mm to (109.2, 96.5)
- moved U2 38.5 mm to (109.9, 87.6)
- moved J3 37.4 mm to (86.4, 94.0)
- moved BT1 34.5 mm to (83.8, 83.8)
- moved C3 32.1 mm to (122.8, 94.6)
- moved Y1 27.0 mm to (118.1, 94.6)
- moved D1 27.0 mm to (122.8, 99.1)
- moved J4 23.4 mm to (110.5, 80.6), turned to 90 degrees
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