File: Arduino Clone - BACEE.kicad_pcb (KiCad board)
At the start: 2 copper layers, 41.9 x 29 mm, 17 parts, among them J1 Digital Pins, J2 Serial, J3 ICSP, J4 I2C, U1 24LC1025, U2 24LC1025, U3 DS13375+, U4 ATMEGA328P-AU, Y1 Crystal 32Mhz, Y2 Crystal 16Mhz

Commit message: Copper Fields - 2 layers
Routing:
- net /Vcc: track 0.00 -> 159.9 mm, vias 0 -> 1
- net GNDPWR: track 0.00 -> 156.5 mm
- net /SCK: track 0.00 -> 111.9 mm, vias 0 -> 2
- net /SDA: track 0.00 -> 61.8 mm, vias 0 -> 1
- net Net-(C1-Pad2): track 0.00 -> 39.6 mm
- net Net-(C2-Pad2): track 0.00 -> 31.5 mm, vias 0 -> 2
- net /RESET: track 0.00 -> 26.1 mm, vias 0 -> 2
- net /MOSI: track 0.00 -> 21.2 mm, vias 0 -> 1
- net /Tx: track 0.00 -> 19.2 mm, vias 0 -> 1
- net /D5: track 0.00 -> 17.2 mm
- net /ADDS1: track 0.00 -> 16.4 mm, vias 0 -> 2
- net /Rx: track 0.00 -> 16.3 mm, vias 0 -> 1
- net /D2: track 0.00 -> 16.1 mm, vias 0 -> 1
- net /MISO: track 0.00 -> 15.7 mm, vias 0 -> 2
- net /ADDS2: track 0.00 -> 15.3 mm
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- added copper zone on B.Cu, net GNDPWR

Commit message: silkscreens
Parts:
- added G***: LOGO, KiCAD_logos:falkon_logo_10.2mm, B.Cu at (104.0, 97.8)
- added REF**: KiCad-Logo2_5mm_SilkScreen, Symbol:KiCad-Logo2_5mm_SilkScreen, B.Cu at (117.6, 92.8)
Other:
- board text added: "Adam Falkowski Designed in NJ"
- board text added: "D2"
- board text added: "D3"
- board text added: "D4"
- board text added: "D5"
- board text added: "D6"
- board text added: "D7"
- board text added: "D8"
- board text added: "GND"
- board text added: "MISO"
- board text added: "MOSI"
- board text added: "RESET"
- board text added: "Rx"
- board text added: "SCK"
- board text added: "SDA"
- board text added: "Tx"
- board text added: "Vcc"
