File: project3_bacee_4_layer.kicad_pcb (KiCad board)
At the start: 2 copper layers, 41.9 x 29 mm, 17 parts, among them J1 Digital Pins, J2 Serial, J3 ICSP, J4 I2C, U1 24LC1025, U2 24LC1025, U3 DS13375+, U4 ATMEGA328P-AU, Y1 Crystal 32Mhz, Y2 Crystal 16Mhz

Commit message: Copper Fields - 2 layers
Routing:
- net /Vcc: track 0.00 -> 157.0 mm
- net GNDPWR: track 0.00 -> 149.0 mm, vias 0 -> 2
- net /SCK: track 0.00 -> 93.0 mm, vias 0 -> 3
- net /SDA: track 0.00 -> 58.1 mm
- net Net-(C2-Pad2): track 0.00 -> 55.5 mm, vias 0 -> 2
- net /RESET: track 0.00 -> 43.4 mm, vias 0 -> 1
- net Net-(C1-Pad2): track 0.00 -> 40.5 mm
- net /D2: track 0.00 -> 29.7 mm, vias 0 -> 1
- net /MOSI: track 0.00 -> 20.8 mm, vias 0 -> 1
- net /D3: track 0.00 -> 20.8 mm, vias 0 -> 1
- net /MISO: track 0.00 -> 18.7 mm, vias 0 -> 1
- net /D5: track 0.00 -> 17.2 mm
- net /Tx: track 0.00 -> 15.8 mm, vias 0 -> 1
- net /ADDS2: track 0.00 -> 15.3 mm
- net /ADDS1: track 0.00 -> 14.6 mm, vias 0 -> 2
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Other:
- copper layers 2 -> 4
